File: pcb/ESP32.kicad_sch (KiCad schematic)
At the start: 33 parts, among them J7 USB_B_Micro, Q1 MMBT3904, Q2 MMBT3904, Q5 BSS138, SW1 RESET, U5 CP2102N-Axx-xQFN24, U6 ESP32-S3-WROOM-1, U9 AP7361C-33E

Commit message: routing start
Parts:
- added R5: 1K, Resistor_SMD:R_0603_1608Metric, symbol Device:R
Connections:
- net OVER_CURRENT: now reaches U6.4 (GPIO4/TOUCH4/ADC1_CH3)
- net at U6.7 (GPIO7/TOUCH7/ADC1_CH6): now also R5.2
- new net USB_ENABLE: R5.1
- no-connect marks 39 -> 37
Changed lines of the file:
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@@
   (no_connect (at 106.68 166.37))
   (no_connect (at 172.72 83.82))
-  (no_connect (at 54.61 54.61))
   (no_connect (at 26.67 168.91))
   (no_connect (at 172.72 58.42))
@@
   (no_connect (at 106.68 163.83))
   (no_connect (at 106.68 176.53))
-  (no_connect (at 54.61 62.23))
   (no_connect (at 172.72 73.66))
   (wire (pts (xy 30.48 57.15) (xy 34.29 57.15))
@@
     (stroke (width 0) (type default) (color 0 0 0 0))
   )
+  (wire (pts (xy 41.91 62.23) (xy 54.61 62.23))
+    (stroke (width 0) (type default) (color 0 0 0 0))
+  )
   (wire (pts (xy 93.98 191.77) (xy 93.98 194.31))
     (stroke (width 0) (type default) (color 0 0 0 0))
@@
     (stroke (width 0) (type default) (color 0 0 0 0))
   )
+  (wire (pts (xy 30.48 54.61) (xy 54.61 54.61))
+    (stroke (width 0) (type default) (color 0 0 0 0))
+  )
   (wire (pts (xy 257.81 153.67) (xy 255.27 153.67))
     (stroke (width 0) (type default) (color 0 0 0 0))
@@
     (stroke (width 0) (type default) (color 0 0 0 0))
   )
+  (wire (pts (xy 30.48 62.23) (xy 34.29 62.23))
+    (stroke (width 0) (type default) (color 0 0 0 0))
+  )
   (wire (pts (xy 132.08 153.67) (xy 132.08 157.48))
     (stroke (width 0) (type default) (color 0 0 0 0))
@@
     (stroke (width 0) (type default) (color 0 0 0 0))
   )
+  (global_label "OVER_CURRENT" (shape input) (at 30.48 54.61 180) (fields_autoplaced)
+    (effects (font (size 1.27 1.27)) (justify right))
+    (property "Intersheet References" "${INTERSHEET_REFS}" (id 0) (at 13.6736 54.5306 0)
+      (effects (font (size 1.27 1.27)) (justify right) hide)
+    )
+  )
   (global_label "U0_TXD" (shape input) (at 109.22 143.51 0) (fields_autoplaced)
     (effects (font (size 1.27 1.27)) (justify left))
@@
     (property "Intersheet References" "${INTERSHEET_REFS}" (id 0) (at 256.4606 28.2483 90)
       (effects (font (size 1.27 1.27)) (justify left) hide)
+    )
+  )
+  (global_label "USB_ENABLE" (shape input) (at 30.48 62.23 180) (fields_autoplaced)
+    (effects (font (size 1.27 1.27)) (justify right))
+    (property "Intersheet References" "${INTERSHEET_REFS}" (id 0) (at 16.274 62.1506 0)
+      (effects (font (size 1.27 1.27)) (justify right) hide)
     )
   )
@@
     (pin "4")
   )
+  (symbol (lib_id "Device:R") (at 38.1 62.23 90) (unit 1)
+    (in_bom yes) (on_board yes)
+    (property "Reference" "R5" (id 0) (at 43.18 60.96 90))
+    (property "Value" "1K" (id 1) (at 46.99 60.96 90))
+    (property "Footprint" "Resistor_SMD:R_0603_1608Metric" (id 2) (at 38.1 64.008 90)
+      (effects (font (size 1.27 1.27)) hide)
+    )
+    (property "Datasheet" "~" (id 3) (at 38.1 62.23 0)
+      (effects (font (size 1.27 1.27)) hide)
+    )
+    (pin "1")
+    (pin "2")
+  )
   (symbol (lib_id "power:GND") (at 49.53 175.26 0) (unit 1)

Commit message: design bugs case update software bugs
Parts:
- renumbered C29 to C1, C20 to C10, C30 to C12, C26 to C14, C28 to C2, C8 to C3, C11 to C4, C25 to C7, C27 to C8, C17 to C9, D2 to D1, D1 to D2, J7 to J4, Q2 to Q1, Q1 to Q4, R13 to R10, R23 to R11, R32 to R13, R31 to R14, R34 to R15, R22 to R16, R36 to R18, R35 to R19, R5 to R3, R1 to R5, R7 to R9, U6 to U2, U5 to U3, U9 to U7
Changed lines of the file:
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@@
   (symbol (lib_id "Device:C") (at 193.04 151.13 180) (unit 1)
     (in_bom yes) (on_board yes)
-    (property "Reference" "C17" (id 0) (at 186.69 152.4 0)
+    (property "Reference" "C9" (id 0) (at 186.69 152.4 0)
       (effects (font (size 1.27 1.27)) (justify right))
     )
@@
   (symbol (lib_id "Device:C") (at 262.89 149.86 270) (unit 1)
     (in_bom yes) (on_board yes)
-    (property "Reference" "C26" (id 0) (at 265.43 146.05 0)
+    (property "Reference" "C14" (id 0) (at 265.43 146.05 0)
       (effects (font (size 1.27 1.27)) (justify left))
     )
@@
   (symbol (lib_id "Device:R") (at 228.6 57.15 0) (mirror y) (unit 1)
     (in_bom yes) (on_board yes)
-    (property "Reference" "R36" (id 0) (at 232.41 55.88 0)
+    (property "Reference" "R18" (id 0) (at 232.41 55.88 0)
       (effects (font (size 1.27 1.27)) (justify left))
     )
@@
   (symbol (lib_id "Interface_USB:CP2102N-Axx-xQFN24") (at 93.98 163.83 0) (unit 1)
     (in_bom yes) (on_board yes)
-    (property "Reference" "U5" (id 0) (at 95.9994 191.77 0)
+    (property "Reference" "U3" (id 0) (at 95.9994 191.77 0)
       (effects (font (size 1.27 1.27)) (justify left))
     )
@@
   (symbol (lib_id "Device:C") (at 245.11 134.62 0) (unit 1)
     (in_bom yes) (on_board yes) (fields_autoplaced)
-    (property "Reference" "C27" (id 0) (at 248.92 133.3499 0)
+    (property "Reference" "C8" (id 0) (at 248.92 133.3499 0)
       (effects (font (size 1.27 1.27)) (justify left))
     )
@@
   (symbol (lib_id "Device:R") (at 57.15 153.67 90) (unit 1)
     (in_bom yes) (on_board yes) (fields_autoplaced)
-    (property "Reference" "R34" (id 0) (at 57.15 147.32 90))
+    (property "Reference" "R15" (id 0) (at 57.15 147.32 90))
     (property "Value" "22K" (id 1) (at 57.15 149.86 90))
     (property "Footprint" "Resistor_SMD:R_0603_1608Metric" (id 2) (at 57.15 155.448 90)
@@
   (symbol (lib_id "Espressif:ESP32-S3-WROOM-1") (at 114.3 69.85 0) (unit 1)
     (in_bom yes) (on_board yes) (fields_autoplaced)
-    (property "Reference" "U6" (id 0) (at 113.665 30.48 0))
+    (property "Reference" "U2" (id 0) (at 113.665 30.48 0))
     (property "Value" "ESP32-S3-WROOM-1" (id 1) (at 113.665 33.02 0))
     (property "Footprint" "Espressif:ESP32-S3-WROOM-1" (id 2) (at 114.3 109.22 0)
@@
   (symbol (lib_id "Device:C") (at 50.8 105.41 0) (unit 1)
     (in_bom yes) (on_board yes)
-    (property "Reference" "C28" (id 0) (at 46.99 102.87 0)
+    (property "Reference" "C2" (id 0) (at 46.99 102.87 0)
       (effects (font (size 1.27 1.27)) (justify left))
     )
@@
   (symbol (lib_id "Transistor_BJT:MMBT3904") (at 138.43 157.48 0) (mirror x) (unit 1)
     (in_bom yes) (on_board yes) (fields_autoplaced)
-    (property "Reference" "Q1" (id 0) (at 143.51 156.2099 0)
+    (property "Reference" "Q4" (id 0) (at 143.51 156.2099 0)
       (effects (font (size 1.27 1.27)) (justify left))
     )
@@
   (symbol (lib_id "Device:R") (at 124.46 146.05 90) (unit 1)
     (in_bom yes) (on_board yes)
-    (property "Reference" "R23" (id 0) (at 124.46 140.97 90))
+    (property "Reference" "R11" (id 0) (at 124.46 140.97 90))
     (property "Value" "10K" (id 1) (at 124.46 143.51 90))
     (property "Footprint" "Resistor_SMD:R_0603_1608Metric" (id 2) (at 124.46 147.828 90)
@@
   (symbol (lib_id "Device:R") (at 214.63 142.24 0) (unit 1)
     (in_bom yes) (on_board yes) (fields_autoplaced)
-    (property "Reference" "R22" (id 0) (at 217.17 140.9699 0)
+    (property "Reference" "R16" (id 0) (at 217.17 140.9699 0)
       (effects (font (size 1.27 1.27)) (justify left))
     )
@@
   (symbol (lib_id "Transistor_BJT:MMBT3904") (at 138.43 142.24 0) (unit 1)
     (in_bom yes) (on_board yes) (fields_autoplaced)
-    (property "Reference" "Q2" (id 0) (at 143.51 140.9699 0)
+    (property "Reference" "Q1" (id 0) (at 143.51 140.9699 0)
       (effects (font (size 1.27 1.27)) (justify left))
     )
@@
   (symbol (lib_id "Device:R") (at 222.25 50.8 90) (unit 1)
     (in_bom yes) (on_board yes) (fields_autoplaced)
-    (property "Reference" "R32" (id 0) (at 222.25 44.45 90))
+    (property "Reference" "R13" (id 0) (at 222.25 44.45 90))
     (property "Value" "1K" (id 1) (at 222.25 46.99 90))
     (property "Footprint" "Resistor_SMD:R_0603_1608Metric" (id 2) (at 222.25 52.578 90)
@@
   (symbol (lib_id "Device:C") (at 49.53 167.64 0) (unit 1)
     (in_bom yes) (on_board yes)
-    (property "Reference" "C25" (id 0) (at 53.34 166.37 0)
+    (property "Reference" "C7" (id 0) (at 53.34 166.37 0)
       (effects (font (size 1.27 1.27)) (justify left))
     )
@@
   (symbol (lib_id "Device:C") (at 267.97 48.26 180) (unit 1)
     (in_bom yes) (on_board yes) (fields_autoplaced)
-    (property "Reference" "C30" (id 0) (at 271.78 46.9899 0)
+    (property "Reference" "C12" (id 0) (at 271.78 46.9899 0)
       (effects (font (size 1.27 1.27)) (justify right))
     )
@@
   (symbol (lib_id "Device:LED") (at 214.63 134.62 270) (unit 1)
     (in_bom yes) (on_board yes) (fields_autoplaced)
-    (property "Reference" "D1" (id 0) (at 217.17 131.7624 90)
+    (property "Reference" "D2" (id 0) (at 217.17 131.7624 90)
       (effects (font (size 1.27 1.27)) (justify left))
     )
@@
   (symbol (lib_id "Diode:1N5819") (at 44.45 153.67 180) (unit 1)
     (in_bom yes) (on_board yes) (fields_autoplaced)
-    (property "Reference" "D2" (id 0) (at 44.7675 147.32 0))
+    (property "Reference" "D1" (id 0) (at 44.7675 147.32 0))
     (property "Value" "1N5819" (id 1) (at 44.7675 149.86 0))
     (property "Footprint" "Diode_SMD:D_SOD-323" (id 2) (at 44.45 149.225 0)
@@
   (symbol (lib_id "Regulator_Linear:AP7361C-33E") (at 203.2 147.32 0) (unit 1)
     (in_bom yes) (on_board yes) (fields_autoplaced)
-    (property "Reference" "U9" (id 0) (at 203.2 139.7 0))
+    (property "Reference" "U7" (id 0) (at 203.2 139.7 0))
     (property "Value" "AP7361C-33E" (id 1) (at 203.2 142.24 0))
     (property "Footprint" "Package_TO_SOT_SMD:SOT-223-3_TabPin2" (id 2) (at 203.2 141.605 0)
@@
   (symbol (lib_id "Device:C") (at 99.06 118.11 90) (unit 1)
     (in_bom yes) (on_board yes)
-    (property "Reference" "C8" (id 0) (at 99.06 114.3 90))
+    (property "Reference" "C3" (id 0) (at 99.06 114.3 90))
     (property "Value" "4.7uF" (id 1) (at 99.06 121.92 90))
     (property "Footprint" "Capacitor_SMD:C_0603_1608Metric" (id 2) (at 102.87 117.1448 0)
@@
   (symbol (lib_id "Device:R") (at 76.2 140.97 90) (unit 1)
     (in_bom yes) (on_board yes)
-    (property "Reference" "R13" (id 0) (at 76.2 138.43 90))
+    (property "Reference" "R10" (id 0) (at 76.2 138.43 90))
     (property "Value" "1K" (id 1) (at 76.2 143.51 90))
     (property "Footprint" "Resistor_SMD:R_0603_1608Metric" (id 2) (at 76.2 142.748 90)
@@
   (symbol (lib_id "Device:C") (at 214.63 151.13 180) (unit 1)
     (in_bom yes) (on_board yes) (fields_autoplaced)
-    (property "Reference" "C20" (id 0) (at 218.44 149.8599 0)
+    (property "Reference" "C10" (id 0) (at 218.44 149.8599 0)
       (effects (font (size 1.27 1.27)) (justify right))
     )
@@
   (symbol (lib_id "Device:R") (at 245.11 124.46 0) (unit 1)
     (in_bom yes) (on_board yes) (fields_autoplaced)
-    (property "Reference" "R31" (id 0) (at 247.65 123.1899 0)
+    (property "Reference" "R14" (id 0) (at 247.65 123.1899 0)
       (effects (font (size 1.27 1.27)) (justify left))
     )
@@
   (symbol (lib_id "Device:C") (at 99.06 128.27 90) (unit 1)
     (in_bom yes) (on_board yes)
-    (property "Reference" "C11" (id 0) (at 99.06 124.46 90))
+    (property "Reference" "C4" (id 0) (at 99.06 124.46 90))
     (property "Value" "0.1uF" (id 1) (at 99.06 132.08 90))
     (property "Footprint" "Capacitor_SMD:C_0603_1608Metric" (id 2) (at 102.87 127.3048 0)
@@
   (symbol (lib_id "Device:C") (at 38.1 105.41 0) (unit 1)
     (in_bom yes) (on_board yes)
-    (property "Reference" "C29" (id 0) (at 34.29 102.87 0)
+    (property "Reference" "C1" (id 0) (at 34.29 102.87 0)
       (effects (font (size 1.27 1.27)) (justify left))
     )
@@
   (symbol (lib_id "Connector:USB_B_Micro") (at 29.21 158.75 0) (unit 1)
     (in_bom yes) (on_board yes) (fields_autoplaced)
-    (property "Reference" "J7" (id 0) (at 29.21 146.05 0))
+    (property "Reference" "J4" (id 0) (at 29.21 146.05 0))
     (property "Value" "USB_B_Micro" (id 1) (at 29.21 148.59 0))
     (property "Footprint" "Connector_USB:USB_Micro-B_Molex-105017-0001" (id 2) (at 33.02 160.02 0)
@@
   (symbol (lib_id "Device:R") (at 38.1 57.15 90) (unit 1)
     (in_bom yes) (on_board yes)
-    (property "Reference" "R1" (id 0) (at 43.18 55.88 90))
+    (property "Reference" "R5" (id 0) (at 43.18 55.88 90))
     (property "Value" "1K" (id 1) (at 46.99 55.88 90))
     (property "Footprint" "Resistor_SMD:R_0603_1608Metric" (id 2) (at 38.1 58.928 90)
@@
   (symbol (lib_id "Device:R") (at 240.03 55.88 0) (mirror y) (unit 1)
     (in_bom yes) (on_board yes)
-    (property "Reference" "R35" (id 0) (at 243.84 54.61 0)
+    (property "Reference" "R19" (id 0) (at 243.84 54.61 0)
       (effects (font (size 1.27 1.27)) (justify left))
     )
@@
   (symbol (lib_id "Device:R") (at 38.1 62.23 90) (unit 1)
     (in_bom yes) (on_board yes)
-    (property "Reference" "R5" (id 0) (at 43.18 60.96 90))
+    (property "Reference" "R3" (id 0) (at 43.18 60.96 90))
     (property "Value" "1K" (id 1) (at 46.99 60.96 90))
     (property "Footprint" "Resistor_SMD:R_0603_1608Metric" (id 2) (at 38.1 64.008 90)
@@
   (symbol (lib_id "Device:R") (at 67.31 147.32 0) (unit 1)
     (in_bom yes) (on_board yes) (fields_autoplaced)
-    (property "Reference" "R7" (id 0) (at 69.85 146.0499 0)
-      (effects (font (size 1.27 1.27)) (justify left))
-    )
+    (property "Reference" "R9" (id 0) (at 69.85 146.0499 0)
+      (effects (font (size 1.27 1.27)) (justify left))
+    )

Commit message: Fix cornerns Add hub diode R3
Parts:
- renumbered C14 to C13, C12 to C15, C8 to C7, C7 to C8, D3 to D4, R19 to R18, R18 to R19, R3 to R2, R4 to R3, R8 to R7
Changed lines of the file:
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@@
   (symbol (lib_id "Device:C") (at 262.89 149.86 270) (unit 1)
     (in_bom yes) (on_board yes)
-    (property "Reference" "C14" (id 0) (at 265.43 146.05 0)
+    (property "Reference" "C13" (id 0) (at 265.43 146.05 0)
       (effects (font (size 1.27 1.27)) (justify left))
     )
@@
   (symbol (lib_id "Device:R") (at 228.6 57.15 0) (mirror y) (unit 1)
     (in_bom yes) (on_board yes)
-    (property "Reference" "R18" (id 0) (at 232.41 55.88 0)
+    (property "Reference" "R19" (id 0) (at 232.41 55.88 0)
       (effects (font (size 1.27 1.27)) (justify left))
     )
@@
   (symbol (lib_id "Device:R") (at 124.46 153.67 90) (unit 1)
     (in_bom yes) (on_board yes)
-    (property "Reference" "R8" (id 0) (at 124.46 156.21 90))
+    (property "Reference" "R7" (id 0) (at 124.46 156.21 90))
     (property "Value" "10K" (id 1) (at 124.46 158.75 90))
     (property "Footprint" "Resistor_SMD:R_0603_1608Metric" (id 2) (at 124.46 155.448 90)
@@
   (symbol (lib_id "Device:C") (at 245.11 134.62 0) (unit 1)
     (in_bom yes) (on_board yes) (fields_autoplaced)
-    (property "Reference" "C8" (id 0) (at 248.92 133.3499 0)
+    (property "Reference" "C7" (id 0) (at 248.92 133.3499 0)
       (effects (font (size 1.27 1.27)) (justify left))
     )
@@
   (symbol (lib_id "Device:C") (at 49.53 167.64 0) (unit 1)
     (in_bom yes) (on_board yes)
-    (property "Reference" "C7" (id 0) (at 53.34 166.37 0)
+    (property "Reference" "C8" (id 0) (at 53.34 166.37 0)
       (effects (font (size 1.27 1.27)) (justify left))
     )
@@
   (symbol (lib_id "Device:C") (at 267.97 48.26 180) (unit 1)
     (in_bom yes) (on_board yes) (fields_autoplaced)
-    (property "Reference" "C12" (id 0) (at 271.78 46.9899 0)
+    (property "Reference" "C15" (id 0) (at 271.78 46.9899 0)
       (effects (font (size 1.27 1.27)) (justify right))
     )
@@
   (symbol (lib_id "Device:R") (at 38.1 59.69 90) (unit 1)
     (in_bom yes) (on_board yes)
-    (property "Reference" "R4" (id 0) (at 43.18 58.42 90))
+    (property "Reference" "R3" (id 0) (at 43.18 58.42 90))
     (property "Value" "1K" (id 1) (at 46.99 58.42 90))
     (property "Footprint" "Resistor_SMD:R_0603_1608Metric" (id 2) (at 38.1 61.468 90)
@@
   (symbol (lib_id "Device:R") (at 240.03 55.88 0) (mirror y) (unit 1)
     (in_bom yes) (on_board yes)
-    (property "Reference" "R19" (id 0) (at 243.84 54.61 0)
+    (property "Reference" "R18" (id 0) (at 243.84 54.61 0)
       (effects (font (size 1.27 1.27)) (justify left))
     )
@@
   (symbol (lib_id "LED:SK6812") (at 256.54 50.8 0) (unit 1)
     (in_bom yes) (on_board yes)
-    (property "Reference" "D3" (id 0) (at 252.73 57.15 0))
+    (property "Reference" "D4" (id 0) (at 252.73 57.15 0))
     (property "Value" "SK6812" (id 1) (at 260.35 57.15 0))
     (property "Footprint" "LED_SMD:LED_SK6812_PLCC4_5.0x5.0mm_P3.2mm" (id 2) (at 257.81 58.42 0)
@@
   (symbol (lib_id "Device:R") (at 38.1 62.23 90) (unit 1)
     (in_bom yes) (on_board yes)
-    (property "Reference" "R3" (id 0) (at 43.18 60.96 90))
+    (property "Reference" "R2" (id 0) (at 43.18 60.96 90))
     (property "Value" "1K" (id 1) (at 46.99 60.96 90))
     (property "Footprint" "Resistor_SMD:R_0603_1608Metric" (id 2) (at 38.1 64.008 90)
