File: pcb/ESP32.kicad_sch (KiCad schematic)
At the start: 34 parts, among them J4 USB_B_Micro, Q1 MMBT3904, Q4 MMBT3904, Q5 BSS138, SW1 RESET, U2 ESP32-S3-WROOM-1, U3 CP2102N-Axx-xQFN24, U7 AP7361C-33E

Commit message: usb resets lower ble advertising reorder references
Parts:
- D1: renamed from D2; footprint Capacitor_SMD:C_0603_1608Metric -> LED_SMD:LED_0603_1608Metric
- renumbered C8 to C10, C13 to C14, C4 to C2, C2 to C3, C3 to C4, C10 to C5, C7 to C6, C9 to C7, D1 to D2, Q4 to Q2, R10 to R1, R2 to R10, R5 to R4, R7 to R5, R9 to R6, R3 to R8, U3 to U1, U7 to U4, U2 to U5
Changed lines of the file:
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@@
   (symbol (lib_id "Device:C") (at 193.04 151.13 180) (unit 1)
     (in_bom yes) (on_board yes)
-    (property "Reference" "C9" (id 0) (at 186.69 152.4 0)
+    (property "Reference" "C7" (id 0) (at 186.69 152.4 0)
       (effects (font (size 1.27 1.27)) (justify right))
     )
@@
   (symbol (lib_id "Device:C") (at 262.89 149.86 270) (unit 1)
     (in_bom yes) (on_board yes)
-    (property "Reference" "C13" (id 0) (at 265.43 146.05 0)
+    (property "Reference" "C14" (id 0) (at 265.43 146.05 0)
       (effects (font (size 1.27 1.27)) (justify left))
     )
@@
   (symbol (lib_id "Interface_USB:CP2102N-Axx-xQFN24") (at 93.98 163.83 0) (unit 1)
     (in_bom yes) (on_board yes)
-    (property "Reference" "U3" (id 0) (at 95.9994 191.77 0)
+    (property "Reference" "U1" (id 0) (at 95.9994 191.77 0)
       (effects (font (size 1.27 1.27)) (justify left))
     )
@@
   (symbol (lib_id "Device:R") (at 124.46 153.67 90) (unit 1)
     (in_bom yes) (on_board yes)
-    (property "Reference" "R7" (id 0) (at 124.46 156.21 90))
+    (property "Reference" "R5" (id 0) (at 124.46 156.21 90))
     (property "Value" "10K" (id 1) (at 124.46 158.75 90))
     (property "Footprint" "Resistor_SMD:R_0603_1608Metric" (id 2) (at 124.46 155.448 90)
@@
   (symbol (lib_id "Device:C") (at 245.11 134.62 0) (unit 1)
     (in_bom yes) (on_board yes) (fields_autoplaced)
-    (property "Reference" "C7" (id 0) (at 248.92 133.3499 0)
+    (property "Reference" "C6" (id 0) (at 248.92 133.3499 0)
       (effects (font (size 1.27 1.27)) (justify left))
     )
@@
   (symbol (lib_id "Espressif:ESP32-S3-WROOM-1") (at 114.3 69.85 0) (unit 1)
     (in_bom yes) (on_board yes) (fields_autoplaced)
-    (property "Reference" "U2" (id 0) (at 113.665 30.48 0))
+    (property "Reference" "U5" (id 0) (at 113.665 30.48 0))
     (property "Value" "ESP32-S3-WROOM-1" (id 1) (at 113.665 33.02 0))
     (property "Footprint" "Espressif:ESP32-S3-WROOM-1" (id 2) (at 114.3 109.22 0)
@@
   (symbol (lib_id "Device:C") (at 50.8 105.41 0) (unit 1)
     (in_bom yes) (on_board yes)
-    (property "Reference" "C2" (id 0) (at 46.99 102.87 0)
+    (property "Reference" "C3" (id 0) (at 46.99 102.87 0)
       (effects (font (size 1.27 1.27)) (justify left))
     )
@@
   (symbol (lib_id "Transistor_BJT:MMBT3904") (at 138.43 157.48 0) (mirror x) (unit 1)
     (in_bom yes) (on_board yes) (fields_autoplaced)
-    (property "Reference" "Q4" (id 0) (at 143.51 156.2099 0)
+    (property "Reference" "Q2" (id 0) (at 143.51 156.2099 0)
       (effects (font (size 1.27 1.27)) (justify left))
     )
@@
   (symbol (lib_id "Device:C") (at 49.53 167.64 0) (unit 1)
     (in_bom yes) (on_board yes)
-    (property "Reference" "C8" (id 0) (at 53.34 166.37 0)
+    (property "Reference" "C10" (id 0) (at 53.34 166.37 0)
       (effects (font (size 1.27 1.27)) (justify left))
     )
@@
   (symbol (lib_id "Device:LED") (at 214.63 134.62 270) (unit 1)
     (in_bom yes) (on_board yes) (fields_autoplaced)
-    (property "Reference" "D2" (id 0) (at 217.17 131.7624 90)
+    (property "Reference" "D1" (id 0) (at 217.17 131.7624 90)
       (effects (font (size 1.27 1.27)) (justify left))
     )
@@
       (effects (font (size 1.27 1.27)) (justify left))
     )
-    (property "Footprint" "Capacitor_SMD:C_0603_1608Metric" (id 2) (at 214.63 134.62 0)
+    (property "Footprint" "LED_SMD:LED_0603_1608Metric" (id 2) (at 214.63 134.62 0)
       (effects (font (size 1.27 1.27)) hide)
     )
@@
   (symbol (lib_id "Diode:1N5819") (at 44.45 153.67 180) (unit 1)
     (in_bom yes) (on_board yes) (fields_autoplaced)
-    (property "Reference" "D1" (id 0) (at 44.7675 147.32 0))
+    (property "Reference" "D2" (id 0) (at 44.7675 147.32 0))
     (property "Value" "1N5819" (id 1) (at 44.7675 149.86 0))
     (property "Footprint" "Diode_SMD:D_SOD-323" (id 2) (at 44.45 149.225 0)
@@
   (symbol (lib_id "Device:R") (at 38.1 59.69 90) (unit 1)
     (in_bom yes) (on_board yes)
-    (property "Reference" "R3" (id 0) (at 43.18 58.42 90))
+    (property "Reference" "R8" (id 0) (at 43.18 58.42 90))
     (property "Value" "1K" (id 1) (at 46.99 58.42 90))
     (property "Footprint" "Resistor_SMD:R_0603_1608Metric" (id 2) (at 38.1 61.468 90)
@@
   (symbol (lib_id "Regulator_Linear:AP7361C-33E") (at 203.2 147.32 0) (unit 1)
     (in_bom yes) (on_board yes) (fields_autoplaced)
-    (property "Reference" "U7" (id 0) (at 203.2 139.7 0))
+    (property "Reference" "U4" (id 0) (at 203.2 139.7 0))
     (property "Value" "AP7361C-33E" (id 1) (at 203.2 142.24 0))
     (property "Footprint" "Package_TO_SOT_SMD:SOT-223-3_TabPin2" (id 2) (at 203.2 141.605 0)
@@
   (symbol (lib_id "Device:C") (at 99.06 118.11 90) (unit 1)
     (in_bom yes) (on_board yes)
-    (property "Reference" "C3" (id 0) (at 99.06 114.3 90))
+    (property "Reference" "C4" (id 0) (at 99.06 114.3 90))
     (property "Value" "4.7uF" (id 1) (at 99.06 121.92 90))
     (property "Footprint" "Capacitor_SMD:C_0603_1608Metric" (id 2) (at 102.87 117.1448 0)
@@
   (symbol (lib_id "Device:R") (at 76.2 140.97 90) (unit 1)
     (in_bom yes) (on_board yes)
-    (property "Reference" "R10" (id 0) (at 76.2 138.43 90))
+    (property "Reference" "R1" (id 0) (at 76.2 138.43 90))
     (property "Value" "1K" (id 1) (at 76.2 143.51 90))
     (property "Footprint" "Resistor_SMD:R_0603_1608Metric" (id 2) (at 76.2 142.748 90)
@@
   (symbol (lib_id "Device:C") (at 214.63 151.13 180) (unit 1)
     (in_bom yes) (on_board yes) (fields_autoplaced)
-    (property "Reference" "C10" (id 0) (at 218.44 149.8599 0)
+    (property "Reference" "C5" (id 0) (at 218.44 149.8599 0)
       (effects (font (size 1.27 1.27)) (justify right))
     )
@@
   (symbol (lib_id "Device:C") (at 99.06 128.27 90) (unit 1)
     (in_bom yes) (on_board yes)
-    (property "Reference" "C4" (id 0) (at 99.06 124.46 90))
+    (property "Reference" "C2" (id 0) (at 99.06 124.46 90))
     (property "Value" "0.1uF" (id 1) (at 99.06 132.08 90))
     (property "Footprint" "Capacitor_SMD:C_0603_1608Metric" (id 2) (at 102.87 127.3048 0)
@@
   (symbol (lib_id "Device:R") (at 38.1 57.15 90) (unit 1)
     (in_bom yes) (on_board yes)
-    (property "Reference" "R5" (id 0) (at 43.18 55.88 90))
+    (property "Reference" "R4" (id 0) (at 43.18 55.88 90))
     (property "Value" "1K" (id 1) (at 46.99 55.88 90))
     (property "Footprint" "Resistor_SMD:R_0603_1608Metric" (id 2) (at 38.1 58.928 90)
@@
   (symbol (lib_id "Device:R") (at 38.1 62.23 90) (unit 1)
     (in_bom yes) (on_board yes)
-    (property "Reference" "R2" (id 0) (at 43.18 60.96 90))
+    (property "Reference" "R10" (id 0) (at 43.18 60.96 90))
     (property "Value" "1K" (id 1) (at 46.99 60.96 90))
     (property "Footprint" "Resistor_SMD:R_0603_1608Metric" (id 2) (at 38.1 64.008 90)
@@
   (symbol (lib_id "Device:R") (at 67.31 147.32 0) (unit 1)
     (in_bom yes) (on_board yes) (fields_autoplaced)
-    (property "Reference" "R9" (id 0) (at 69.85 146.0499 0)
-      (effects (font (size 1.27 1.27)) (justify left))
-    )
+    (property "Reference" "R6" (id 0) (at 69.85 146.0499 0)
+      (effects (font (size 1.27 1.27)) (justify left))
+    )
