File: pcb/EasyKVM.kicad_pcb (KiCad board)
At the start: 4 copper layers, 75 x 75 mm, 62 parts, among them J1 USB_B_Micro, J2 USB_B_Micro, J3 HDMI_A, J4 USB_B_Micro, J5 HDMI_A, J6 USB_A, J7 USB_A, Q1 MMBT3904, Q2 BSS138, Q3 BSS138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

Commit message: usb resets lower ble advertising reorder references
Parts:
- D1: renamed from D2; footprint Capacitor_SMD:C_0603_1608Metric -> LED_SMD:LED_0603_1608Metric
- renumbered C8 to C10, C12 to C11, C11 to C12, C14 to C13, C13 to C14, C4 to C2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
